Commit message: Aggiornamento_15_11

File: description/robot.urdf.xacro (robot description, xacro)
@@ -3,3 +3,4 @@
     <xacro:include filename="robot_core.xacro" />
     <xacro:include filename="inertial_macros.xacro" />
+    <xacro:include filename="gazebo_control.xacro" />
 </robot>

File: description/robot_core.xacro (robot description, xacro)
@@ -63,4 +63,9 @@
         <origin xyz="0 0 0" rpy="0 0 0"/>
     </xacro:inertial_cylinder>
+    <gazebo>
+    <material>Gazebo/Black</material>
+        <mu1 value="0.01"/>
+        <mu2 value="0.01"/>
+    </gazebo>
 </link>
 <!-- RIGHT WHEEL -->
@@ -87,4 +92,9 @@
         <origin xyz="0 0 0" rpy="0 0 0"/>
     </xacro:inertial_cylinder>
+    <gazebo>
+    <material>Gazebo/Black</material>
+        <mu1 value="0.01"/>
+        <mu2 value="0.01"/>
+    </gazebo>
 </link>
 <!-- CASTER WHEEL -->
@@ -111,3 +121,8 @@
     </xacro:inertial_sphere>
 </link>
+<gazebo reference="caster_wheel">
+     <material>Gazebo/Black</material>
+        <mu1 value="0.01"/>
+        <mu2 value="0.01"/>
+    </gazebo>
 </robot>
