Commit message: aggiunta_lidar

File: description/robot_core.xacro (robot description, xacro)
@@ -13,4 +13,7 @@
 <material name="black">
     <color rgba="0 0 0 1"/>
+</material>
+<material name="red">
+    <color rgba="1 0 0 1"/>
 </material>
 <link name="base_link">
@@ -64,8 +67,4 @@
     </xacro:inertial_cylinder>
     <gazebo>
-    <material>Gazebo/Black</material>
-        <mu1 value="0.01"/>
-        <mu2 value="0.01"/>
-    </gazebo>
 </link>
 <!-- RIGHT WHEEL -->

Commit message: modifiche_4_12_2

File: description/robot_core.xacro (robot description, xacro)
@@ -17,5 +17,14 @@
     <color rgba="1 0 0 1"/>
 </material>
+    <!--BASE LINK-->
 <link name="base_link">
+</link>
+    <!--BASE FOOTPRINT-->
+<joint name="base_footprint_joint" type="fixed">
+    <parent link="base_link"/>
+    <child link="base_footprint"/>
+    <origin xyz="0 0 0" rpy="0 0 0"/>
+</joint>
+<link name="base_footprint">
 </link>
     <!--CHASSIS-->
